Commit message: update

File: hercules/urdf/finished.urdf.xacro (robot description, xacro)
@@ -28,9 +28,10 @@
     <inertial>
         <origin xyz="0 0 0" rpy="0 0 0"/>
-        <mass value="1.8"/>
-        <inertia
-          ixx="0.0029" ixy="0" ixz="0"
-          iyy="0.0065" iyz="0"
-          izz="0.0091"/>
+       <mass value="16.523"/>
+      <!-- Moments of inertia: ( chassis without wheels ) -->
+      <inertia
+        ixx="0.3136" ixy="-0.0008" ixz="0.0164"
+        iyy="0.3922" iyz="-0.0009"
+        izz="0.4485"/>
     </inertial>
   </link>
@@ -38,4 +39,10 @@
       <material>Gazebo/Green</material>
   </gazebo>
+  <!-- https://answers.ros.org/question/151121/how-to-create-soft-objects-wheel-tires-in-gazebo/?answer=197040#post-id-197040 -->
+  <xacro:macro name="cylinder_inertia" params="m r h">
+    <inertia  ixx="${m*(3*r*r+h*h)/12}" ixy = "0" ixz = "0"
+            iyy="${m*(3*r*r+h*h)/12}" iyz = "0"
+            izz="${m*r*r/2}" />
+  </xacro:macro>
   <xacro:macro name="wheel" params="prefix *joint_pose">
     <link name="${prefix}_wheel">
@@ -55,9 +62,6 @@
       <inertial>
         <origin xyz="0 0 0" rpy="0 0 0"/>
-        <mass value="0.05"/>
-        <inertia
-          ixx="2.6326e-5" ixy="0" ixz="0"
-          iyy="4.5156e-5" iyz="0"
-          izz="2.6326e-5"/>
+        <mass value="0.5"/>
+        <cylinder_inertia  m="0.5" r="${wheel_radius}" h="${wheel_width}" />
       </inertial>
     </link>
@@ -74,5 +78,5 @@
       <type>transmission_interface/SimpleTransmission</type>
       <joint name="${prefix}_wheel_joint">
-        <hardwareInterface>VelocityJointInterface</hardwareInterface>
+        <hardwareInterface>hardware_interface/VelocityJointInterface</hardwareInterface>
       </joint>
       <actuator name="${prefix}_actuator">
@@ -93,4 +97,29 @@
     <origin xyz="${-wheelbase/2} ${-track/2} ${wheel_vertical_offset}" rpy="0 0 0" />
   </xacro:wheel>
+<link name="laser_link">
+    <collision>
+      <origin xyz="0 0 0" rpy="0 0 0"/>
+      <geometry>
+        <box size="0.05 0.05 0.06"/>
+      </geometry>
+    </collision>
+    <visual>
+      <origin xyz="0 0 0" rpy="0 0 0"/>
+      <geometry>
+        <box size="0.05 0.05 0.05"/>
+      </geometry>
+    </visual>
+    <inertial>
+      <mass value="1e-5" />
+      <origin xyz="0 0 0" rpy="0 0 0"/>
+      <inertia ixx="1e-6" ixy="0" ixz="0" iyy="1e-6" iyz="0" izz="1e-6" />
+    </inertial>
+  </link>
+  <joint name="laser_joint" type="fixed">
+    <axis xyz="0 1 0" />
+    <origin xyz="0 0 0.0475" rpy="0 0 0"/>
+    <parent link="base_link"/>
+    <child link="laser_link"/>
+  </joint>
    <!-- Gazebo plugin for control using diff_drive_controller -->
   <gazebo>
@@ -100,3 +129,34 @@
   </gazebo>
   <!-- Gazebo -->
+  <gazebo reference="laser_link">
+    <sensor type="gpu_ray" name="laser">
+      <pose>0 0 0 0 0 0</pose>
+      <visualize>false</visualize>
+      <update_rate>40</update_rate>
+      <ray>
+        <scan>
+          <horizontal>
+            <samples>720</samples>
+            <resolution>1</resolution>
+            <min_angle>-${PI/2}</min_angle>
+            <max_angle>${PI/2}</max_angle>
+          </horizontal>
+        </scan>
+        <range>
+          <min>0.10</min>
+          <max>30.0</max>
+          <resolution>0.01</resolution>
+        </range>
+        <noise>
+          <type>gaussian</type>
+          <mean>0.0</mean>
+          <stddev>0.01</stddev>
+        </noise>
+      </ray>
+      <plugin name="gpu_laser" filename="libgazebo_ros_gpu_laser.so">
+        <topicName>scan</topicName>
+        <frameName>laser_link</frameName>
+      </plugin>
+    </sensor>
+  </gazebo>
 </robot>

File: hercules/urdf/hercules.urdf.xacro (robot description, xacro)
@@ -29,9 +29,10 @@
     <inertial>
     <origin xyz="0 0 0" rpy="0 0 0"/>
-    <mass value="1.8"/>
-    <inertia
-        ixx="0.0029" ixy="0" ixz="0"
-        iyy="0.0065" iyz="0"
-        izz="0.0091"/>
+     <mass value="16.523"/>
+      <!-- Moments of inertia: ( chassis without wheels ) -->
+      <inertia
+        ixx="0.3136" ixy="-0.0008" ixz="0.0164"
+        iyy="0.3922" iyz="-0.0009"
+        izz="0.4485"/>
     </inertial>
   </link>
@@ -40,4 +41,10 @@
    <material>Gazebo/Green</material>
   </gazebo>
+   <!-- https://answers.ros.org/question/151121/how-to-create-soft-objects-wheel-tires-in-gazebo/?answer=197040#post-id-197040 -->
+  <xacro:macro name="cylinder_inertia" params="m r h">
+    <inertia  ixx="${m*(3*r*r+h*h)/12}" ixy = "0" ixz = "0"
+            iyy="${m*(3*r*r+h*h)/12}" iyz = "0"
+            izz="${m*r*r/2}" />
+  </xacro:macro>
   <!-- wheels goes below -->
   <xacro:macro name="wheel" params="prefix *joint_pose">
@@ -59,10 +66,6 @@
         <inertial>
         <origin xyz="0 0 0" rpy="0 0 0"/>
-        <mass value="0.05"/>
-        <inertia
-            ixx="2.6326e-5" ixy="0" ixz="0"
-            iyy="4.5156e-5" iyz="0"
-            izz="2.6326e-5"/>
-        </inertial>
+        <mass value="0.5"/>
+        <cylinder_inertia  m="0.05" r="${wheel_radius}" h="${wheel_width}" />
     </link>
     <!-- Joint -->
@@ -99,4 +102,6 @@
   </xacro:wheel>
   <!-- wheel links goes above -->
+  <!-- laser link and joint goes below -->
+  <!-- laser link and joint goes above -->
   <!-- Gazebo plugin for control using diff_drive_controller -->
   <gazebo>
@@ -106,3 +111,5 @@
   </gazebo>
   <!-- Gazebo -->
+  <!-- Gazebo plugin for laser scanner -->
+  <!-- Gazebo -->
 </robot>
